Commit message: Added URDF for the arena Created a URDF file for the arena itself. Also added textures and collisions to it. Tested loading into PyBullet and it worked well.

File: pybullet_prototype/data/ArenaLayout/ArenaLayout.urdf (robot description, URDF)
Before this commit: robot ArenaLayout.urdf, 1 links, 0 joints
Links:
- removed link baseLink
- added link Arena; collision box size=0.01905 0.3048 0.0381; collision box size=0.01905 0.3048 0.0381
