Commit message: Changed units to metric and removed collision

File: data/button/button.urdf (robot description, URDF)
Before this commit: robot button, 3 links, 2 joints
Links:
- link base_link: mass None -> .005; geometry collision cylinder length=0.0286 radius=0.014; visual cylinder length=0.0286 radius=0.014
- link push_link: mass None -> .005; geometry collision cylinder length=0.0097 radius=0.011325; visual cylinder length=0.0097 radius=0.011325
- link ring_link: mass None -> .005; geometry collision cylinder length=0.0047 radius=0.01665; visual cylinder length=0.0047 radius=0.01665
Joints:
- joint ring_joint: limit lower=-4.1 upper=0 effort=0.2 velocity=0.5 -> lower=-0.0041 upper=0 effort=0.2 velocity=0.5

File: data/field/field.urdf (robot description, URDF)
Before this commit: robot field.urdf, 1 links, 0 joints
Links:
- link field_link: mass None -> 1e10
