Commit message: Increased the force limit for the racecar and fixed typos

File: data/racecar/racecar.urdf (robot description, URDF)
Before this commit: robot racecar, 13 links, 12 joints
Joints:
- joint left_rear_wheel_joint: limit effort=10 velocity=100 -> effort=10000 velocity=100
- joint left_steering_hinge_joint: limit lower=-1.0 upper=1.0 effort=10 velocity=100 -> lower=-1.0 upper=1.0 effort=10000 velocity=100
- joint right_rear_wheel_joint: limit effort=10 velocity=100 -> effort=10000 velocity=100
- joint right_steering_hinge_joint: limit lower=-1.0 upper=1.0 effort=10 velocity=100 -> lower=-1.0 upper=1.0 effort=10000 velocity=100
