Commit message: Initial test of lego block

File: data/lego/lego.urdf (robot description, URDF)
Before this commit: robot lego, 18 links, 17 joints
Links:
- removed link back_panel
- removed link bl_brace
- removed link bl_stud
- removed link br_brace
- removed link br_stud
- removed link cen_stud
- removed link fl_brace
- removed link fl_stud
- removed link fr_brace
- removed link fr_stud
- removed link front_panel
- removed link lb_brace
- removed link left_panel
- removed link lf_brace
- removed link rb_brace
- removed link rf_brace
- removed link right_panel
- removed link top_panel
- added link block, mass 0.005762631744; collision box size=0.00131 0.00168 0.0169; collision box size=0.00131 0.00168 0.0169
Joints:
- removed joint top_back
- removed joint top_bbl
- removed joint top_bbr
- removed joint top_bfl
- removed joint top_bfr
- removed joint top_bl
- removed joint top_blb
- removed joint top_blf
- removed joint top_br
- removed joint top_brb
- removed joint top_brf
- removed joint top_cen
- removed joint top_fl
- removed joint top_fr
- removed joint top_front
- removed joint top_left
- removed joint top_right

Commit message: Finished making the lego XACRO Right now I don't have the exact inertia matrix, so I just approximated the lego as a cube. They seem to stick well with collisionStiffness at 1e6 and collisionDamping at 1e5. We will need to tune these values, though.

File: data/lego/lego.urdf (robot description, URDF)
Before this commit: robot lego, 1 links, 0 joints
Links:
- link block: mass 0.005762631744 -> 0.088400371684

File: data/lego/lego.xacro (robot description, xacro)
@@ -5,6 +5,4 @@
         <color rgba="1 1 1 1"/>
     </material>
-    <!-- Desnity for mass calculations -->
-    <xacro:property name="density" value="4000"/> <!-- kg/m^3 -->
     <!-- Macro for visual and collision boxes -->
     <!-- Length, width, and height are along X, Y, and Z -->
@@ -26,13 +24,4 @@
                              l="${l}" w="${w}" h="${h}"/>
         </collision>
-        <inertial>
-            <xacro:property name="m" value="${density*l*w*h}"/>
-            <origin rpy="0 0 0" xyz="${x} ${y} ${z}"/>
-            <mass value="${m}"/>
-            <inertia ixx="${1/12 * m * (w*w + h*h)}"
-                     iyy="${1/12 * m * (l*l + h*h)}"
-                     izz="${1/12 * m * (l*l + w*w)}"
-                     ixy="0" ixz="0" iyz="0"/>
-        </inertial>
     </xacro:macro>
     <!-- Macro for visual and collision cylinders -->
@@ -53,12 +42,4 @@
             <xacro:cyl_inner x="${x}" y="${y}" z="${z}" r="${r}" l="${l}"/>
         </collision>
-        <inertial>
-            <xacro:property name="m" value="${density*pi*r*r*l}"/>
-            <mass value="${m}"/>
-            <inertia ixx="${1/12 * m * (3*r*r + l*l)}"
-                     iyy="${1/12 * m * (3*r*r + l*l)}"
-                     izz="${1/2 * m * r*r}"
-                     ixy="0" ixz="0" iyz="0"/>
-        </inertial>
     </xacro:macro>
     <link name="block">
@@ -99,4 +80,14 @@
         <xacro:pri x="-.00799" y="-.013535" z=".00845"
                    l=".00131"  w=".00168"   h=".0169"/>
+        <!-- Inertia is an approximation for now -->
+        <inertial>
+            <origin rpy="0 0 0" xyz="0 0 ${.02209/2}"/>
+            <xacro:property name="m" value="${4000 * .03163 * .03163 * .02209}"/>
+            <mass value="${m}"/>
+            <inertia ixx="${1/12 * m * (.03163*.03163 + .02209*.02209)}"
+                     iyy="${1/12 * m * (.03163*.03163 + .02209*.02209)}"
+                     izz="${1/12 * m * (2*.03163*.03163)}"
+                     ixy="0" ixz="0" iyz="0"/>
+        </inertial>
     </link>
 </robot>
