Commit message: Lowercased modules, Renamed ArenaLayout to field, removed commented code.

File: data/field/field.urdf (robot description, URDF)
Before this commit: robot ArenaLayout.urdf, 1 links, 0 joints
Links:
- removed link Arena
- added link field_link; collision box size=0.01905 0.3048 0.0381; collision box size=0.01905 0.3048 0.0381

Commit message: Started consolidating the field URDF I found that having ten different URDFs for the buttons then making calls to PyBullet for each one slowed things down dramatically. Thus, I began consolidating the buttons into a single URDF and updating the code to reflect that. The code in this state works but is nonetheless unclean.

File: data/field/field.urdf (robot description, URDF)
Before this commit: robot field.urdf, 1 links, 0 joints
Links:
- added link push_link_0, mass .005; collision cylinder length=0.0097 radius=0.011325; visual cylinder length=0.0097 radius=0.011325
- added link push_link_1, mass .005; collision cylinder length=0.0097 radius=0.011325; visual cylinder length=0.0097 radius=0.011325
- added link push_link_2, mass .005; collision cylinder length=0.0097 radius=0.011325; visual cylinder length=0.0097 radius=0.011325
- added link push_link_3, mass .005; collision cylinder length=0.0097 radius=0.011325; visual cylinder length=0.0097 radius=0.011325
- added link push_link_4, mass .005; collision cylinder length=0.0097 radius=0.011325; visual cylinder length=0.0097 radius=0.011325
- added link push_link_5, mass .005; collision cylinder length=0.0097 radius=0.011325; visual cylinder length=0.0097 radius=0.011325
- added link push_link_6, mass .005; collision cylinder length=0.0097 radius=0.011325; visual cylinder length=0.0097 radius=0.011325
- added link push_link_7, mass .005; collision cylinder length=0.0097 radius=0.011325; visual cylinder length=0.0097 radius=0.011325
- added link push_link_8, mass .005; collision cylinder length=0.0097 radius=0.011325; visual cylinder length=0.0097 radius=0.011325
- added link push_link_9, mass .005; collision cylinder length=0.0097 radius=0.011325; visual cylinder length=0.0097 radius=0.011325
- added link ring_link_0, mass .005; collision cylinder length=0.0047 radius=0.01665; visual cylinder length=0.0047 radius=0.01665
- added link ring_link_1, mass .005; collision cylinder length=0.0047 radius=0.01665; visual cylinder length=0.0047 radius=0.01665
- added link ring_link_2, mass .005; collision cylinder length=0.0047 radius=0.01665; visual cylinder length=0.0047 radius=0.01665
- added link ring_link_3, mass .005; collision cylinder length=0.0047 radius=0.01665; visual cylinder length=0.0047 radius=0.01665
- added link ring_link_4, mass .005; collision cylinder length=0.0047 radius=0.01665; visual cylinder length=0.0047 radius=0.01665
- added link ring_link_5, mass .005; collision cylinder length=0.0047 radius=0.01665; visual cylinder length=0.0047 radius=0.01665
- added link ring_link_6, mass .005; collision cylinder length=0.0047 radius=0.01665; visual cylinder length=0.0047 radius=0.01665
- added link ring_link_7, mass .005; collision cylinder length=0.0047 radius=0.01665; visual cylinder length=0.0047 radius=0.01665
- added link ring_link_8, mass .005; collision cylinder length=0.0047 radius=0.01665; visual cylinder length=0.0047 radius=0.01665
- added link ring_link_9, mass .005; collision cylinder length=0.0047 radius=0.01665; visual cylinder length=0.0047 radius=0.01665
Joints:
- added joint field_ring_joint_0: type fixed, parent field_link, child ring_link_0
- added joint field_ring_joint_1: type fixed, parent field_link, child ring_link_1
- added joint field_ring_joint_2: type fixed, parent field_link, child ring_link_2
- added joint field_ring_joint_3: type fixed, parent field_link, child ring_link_3
- added joint field_ring_joint_4: type fixed, parent field_link, child ring_link_4
- added joint field_ring_joint_5: type fixed, parent field_link, child ring_link_5
- added joint field_ring_joint_6: type fixed, parent field_link, child ring_link_6
- added joint field_ring_joint_7: type fixed, parent field_link, child ring_link_7
- added joint field_ring_joint_8: type fixed, parent field_link, child ring_link_8
- added joint field_ring_joint_9: type fixed, parent field_link, child ring_link_9
- added joint ring_push_joint_0: type prismatic, parent ring_link_0, child push_link_0, axis 1 0 0, limit lower=-0.0041 upper=0 effort=0.2 velocity=0.5
- added joint ring_push_joint_1: type prismatic, parent ring_link_1, child push_link_1, axis 1 0 0, limit lower=-0.0041 upper=0 effort=0.2 velocity=0.5
- added joint ring_push_joint_2: type prismatic, parent ring_link_2, child push_link_2, axis 1 0 0, limit lower=-0.0041 upper=0 effort=0.2 velocity=0.5
- added joint ring_push_joint_3: type prismatic, parent ring_link_3, child push_link_3, axis 1 0 0, limit lower=-0.0041 upper=0 effort=0.2 velocity=0.5
- added joint ring_push_joint_4: type prismatic, parent ring_link_4, child push_link_4, axis 1 0 0, limit lower=-0.0041 upper=0 effort=0.2 velocity=0.5
- added joint ring_push_joint_5: type prismatic, parent ring_link_5, child push_link_5, axis 1 0 0, limit lower=-0.0041 upper=0 effort=0.2 velocity=0.5
- added joint ring_push_joint_6: type prismatic, parent ring_link_6, child push_link_6, axis 1 0 0, limit lower=-0.0041 upper=0 effort=0.2 velocity=0.5
- added joint ring_push_joint_7: type prismatic, parent ring_link_7, child push_link_7, axis 1 0 0, limit lower=-0.0041 upper=0 effort=0.2 velocity=0.5
- added joint ring_push_joint_8: type prismatic, parent ring_link_8, child push_link_8, axis 1 0 0, limit lower=-0.0041 upper=0 effort=0.2 velocity=0.5
- added joint ring_push_joint_9: type prismatic, parent ring_link_9, child push_link_9, axis 1 0 0, limit lower=-0.0041 upper=0 effort=0.2 velocity=0.5

Commit message: Pushed the buttons into the wall Changed the collision for the field to allow square indents around the buttons. Also changed the model to reflect this.

File: data/field/field.urdf (robot description, URDF)
Before this commit: robot field.urdf, 21 links, 20 joints
Links:
- link field_link: mass 1e10 -> None; geometry collision box size=0.0153875 0.075 0.0333; collision box size=0.0153875 0.0762 0.0333

Commit message: Revert "Merge pull request #30 from binitshah/master"
This reverts commit 2c39b231fde2b15822e78cb593547899e79a0da3, reversing
changes made to 7f9655104f20b6233fcf08c52ae4a30daa0776f1.

File: data/field/field.urdf (robot description, URDF)
Before this commit: robot field.urdf, 21 links, 20 joints
Links:
- link field_link: mass 0.024 -> None
