Commit message: Blockstacker URDF improvements

File: data/blockstacker/urdf/blockstacker.urdf (robot description, URDF)
Before this commit: robot blockstacker, 20 links, 19 joints
Links:
- link enable_button_link: mass None -> 0.024
- link left_camera_link: geometry collision mesh filename=../meshes/left_camera_link.STL scale=0.001 0.001 0.001; visual mesh filename=../meshes/left_camera_link.STL scale=0.001 0.001 0.001
- link right_camera_link: geometry collision mesh filename=../meshes/right_camera_link.STL scale=0.001 0.001 0.001; visual mesh filename=../meshes/right_camera_link.STL scale=0.001 0.001 0.001
Joints:
- joint left_camera_joint: origin xyz=0.015 0.0275000000000001 -0.001451698777701 rpy=-1.5707963267949 0 3.14159265358978 -> xyz=0.0276 0.0371 0.002 rpy=-1.5707963267949 0 3.14159265358978
- joint right_camera_joint: origin xyz=0.0150000000000001 0.0275000000000002 -0.001451698777701 rpy=-1.5707963267949 0 3.14159265358978 -> xyz=0.0276 0.0371 0.002 rpy=-1.5707963267949 0 3.14159265358978

Commit message: updated lego simulation and added differentialdrive abstraction

File: data/blockstacker/urdf/blockstacker.urdf (robot description, URDF)
Before this commit: robot blockstacker, 20 links, 19 joints
Links:
- link base_link: geometry collision mesh filename=../meshes/base_link.obj; visual mesh filename=../meshes/base_link.STL
